File: STM32 control board.sch (EAGLE design)
At the start: 104 parts, among them J1 PJ-063BH, J10 S10B-PH, J11 S10B-PH, J12 S10B-PH, J13 S10B-PH, J14 S3B-PH, J15 S3B-PH, J16 S3B-PH, J17 S3B-PH, J2 S4B-PH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

Commit message: Update STM32 control board.sch
Review
Parts:
- added D6: Green, Semiconductor_devices:LED0805
- added R18: Calc_needed, Resistors:R-EU0402
- C1: device Capacitors:C-EU1206 -> Capacitors:C-EU-CERAMIC1206
- C2: device Capacitors:C-EU0805 -> Capacitors:C-EU-CERAMIC0805
- C3, C4, C5, C6: device Capacitors:C-EU0402 -> Capacitors:C-EU-CERAMIC0402
- J7: value (none) -> black
- TP1: value TEST_RING -> (none)
- U2: value INA240A1 -> (none)
- renumbered U12 to U2
Connections:
- removed net PC15: U10A.PC15-OSC32_OUT
- new net N$7: D6.A, R18.1
- net +3V3: now also R18.2
- net GND: now also D6.C
