File: STM32 control board.sch (EAGLE design)
At the start: 106 parts, among them J1 PJ-063BH, J10 S10B-PH, J11 S10B-PH, J12 S10B-PH, J13 S10B-PH, J14 S3B-PH, J15 S3B-PH, J16 S3B-PH, J17 S3B-PH, J2 S4B-PH, J3 S3B-PH, J4 S3B-PH, J55 S2B-PH, J65 S2B-PH, J7 black, J8 S6B-PH, J9 S4B-PH, U1 TPS7A19, U10 STM32G474, U11 DRV8701VIA, U5 REF3330, U6 REF3318, U7 TCAN1042HGV, U8 ICM_20600, X1 CSTNE

Commit message: power_output_design_in_progress
Parts:
- added C17: 100uF, Capacitors:C-EU-CERAMIC0402
- added C7, C8: 47uF, Capacitors:C-EU-CERAMIC1210
- added C9: 10uF, Capacitors:C-EU-CERAMIC1206
- added D5: SMC-SCHOTTKY, Semiconductor_devices:SMC-SCHOTTKY
- added R19: 10k, Resistors:R-EU0402
- added SW1: DP3T-1-1825289-0, buttons and switches:DP3T-1-1825289-0
- added U$1: DG301-4P, Terminal blocks:DG301-4P
- added U3: L2293Q, Transistors drivers:L2293Q
Connections:
- new net N$10: SW1.3, SW1.7
- new net N$12: SW1.4, SW1.8
- new net N$13: D5.A, SW1.2, SW1.6
- new net N$14: C17.1, C7.1, C8.1, C9.1, D5.C, R19.2, U3.VS, U3.VS@1
- new net N$9: SW1.1, SW1.5
- net GND: now also C17.2, C7.2, C8.2, C9.2, R19.1

Commit message: Update STM32 control board.sch
Parts:
- removed C45, C46: (no value), Capacitors:C-EU-ELECTROLYTICH6.1
- removed R1: 10k, Resistors:R-EU0402
- removed U$1: DG301-4P, Terminal blocks:DG301-4P
- added C31: 100nF, Capacitors:C-EU-CERAMIC0402
- added C32, C33, C34: 47uF, Capacitors:C-EU-CERAMIC1210
- added C35, C36: 10uF, Capacitors:C-EU-CERAMIC1206
- added GND, VIN: (no value), testing:TEST_RING
- added J18: DG301-4P, Terminal blocks:DG301-4P
- added R20, R21, R22, R23, R24, R25: 100, Resistors:R-EU0402
- C17: value 100uF -> 100nF
- C2: value 22uF -> 47uF; device Capacitors:C-EU-CERAMIC0805 -> Capacitors:C-EU-CERAMIC1210; MANUFACTURER_PART_NUMBER (none) -> GRM32ER61C476ME15L
- C7, C8: MANUFACTURER_PART_NUMBER (none) -> GRM32ER61C476ME15L
- C9: MANUFACTURER_PART_NUMBER (none) -> CL31B106KOHNNNE
- D5: value SMC-SCHOTTKY -> SMC-SCHOTTKYSMC; device Semiconductor_devices:SMC-SCHOTTKY -> Semiconductor_devices:SMC-SCHOTTKYSMC; MANUFACTURER_PART_NUMBER (none) -> B520C-13-F
- Q1, Q2, Q3, Q4: device Transistors:SON5X6_MOSFET -> Transistors:CSD15571Q2
- R11: device Resistors:R_EU_CS1206 -> Resistors:R_EU_CS; MANUFACTURER_PART_NUMBER (none) -> STE0805MW75R010F
- U2: MANUFACTURER_PART_NUMBER (none) -> INA240
- renumbered TP1 to 5V
Connections:
- removed net N$10: SW1.3, SW1.7
- removed net N$12: SW1.4, SW1.8
- removed net N$22: R1.1, U1.DELAY
- removed net N$9: SW1.1, SW1.5
- removed net PA10: U10A.PA10
- removed net PA11: U10A.PA11
- removed net PA8: U10A.PA8
- removed net PA9: U10A.PA9
- new net BRIDGE1_EN: R24.1, U10B.PF9
- new net BRIDGE2_EN: R25.1, U10B.PF10
- new net N$15: R22.2, U3.IN2
- new net N$16: R21.2, U3.IN3
- new net N$17: C31.1, U3.VSS
- new net N$18: R20.2, U3.IN4
- new net N$19: R24.2, U3.EN1
- new net N$20: R25.2, U3.EN2
- new net N$8: R23.2, U3.IN1
- new net POUT1: J18.1, U3.OUT1
- new net POUT2: J18.2, U3.OUT2
- new net POUT3: J18.3, U3.OUT3
- new net POUT4: J18.4, U3.OUT4
- new net POWER_OUT1: R23.1, U10A.PA8
- new net POWER_OUT2: R22.1, U10A.PA9
- new net POWER_OUT3: R21.1, U10A.PA10
- new net POWER_OUT4: R20.1, U10A.PA11
- net +3V3: now also SW1.1, SW1.5
- net +5V: now also SW1.3, SW1.7; no longer R1.2
- net GND: now also C31.2, C33.2, C34.2, C35.2, C36.2, GND.P$1, Q4.S, U3.GND, U3.GND@1, U3.GND@2, U3.GND@3, U3.GND@4, U3.NC1@2, U3.NC1@3, U3.NC1@4, U3.NC1@5, U3.NC1@6, U3.NC1@7, U3.NC1@8, U3.NC2@1, U3.NC2@18, U3.NC2@19, U3.NC2@20, U3.NC2@21, U3.NC2@22, U3.NC2@23; no longer C45.-, C46.-, Q2.S
- net M_GH2: now also Q2.G; no longer Q4.G
- net M_GL1: now also Q4.G; no longer Q2.G
- net M_SH1: now also Q4.D; no longer Q2.D
- net M_SH2: now also Q2.S; no longer Q4.S
- net VBAT: now also C33.1, C34.1, C35.1, C36.1, Q2.D; no longer C45.+, C46.+, C47.1, C49.1, C50.1, Q4.D, U11.VM
- net VDD: now also C47.1, C49.1, C50.1, SW1.4, SW1.8, U11.VM, VIN.P$1
Other:
- note added: "25V"
- note removed: "50V"
- moved on the sheet: C17, C7, C8, C9, D5, R19, SW1, U3, X1

Commit message: board created
Parts:
- removed C15, C16: 100nF, Capacitors:C-EU-CERAMIC0402
- removed C32: 47uF, Capacitors:C-EU-CERAMIC1210
- removed D5: SMC-SCHOTTKYSMC, Semiconductor_devices:SMC-SCHOTTKYSMC
- removed J55, J65: S2B-PH, con-jst-ph:S2B-PH
- removed J7: black, Terminal blocks:SCREW_TERMINAL_2P_ALTERNATIVE
- removed J9: S4B-PH, con-jst-ph:S4B-PH
- removed R19: 10k, Resistors:R-EU0402
- removed R6: 120, Resistors:R-EU0805
- removed SW1: DP3T-1-1825289-0, buttons and switches:DP3T-1-1825289-0
- removed TP12: RX, testing:TEST_RING
- removed TP9: TX, testing:TEST_RING
- removed U7: TCAN1042HGV, texas Instrumets:8_PIN_CAN_TRANSIVERSTB_VIO
- added J5: S6B-PH, con-jst-ph:S6B-PH
- S1: value (none) -> B3F-4055; device buttons and switches:MOMENTARY-SWITCH-SPST-2-[SMD-5.2MM] -> buttons and switches:B3F-4055
Connections:
- removed net +5V: 5V.P$1, C15.1, C2.1, R2.2, SW1.3, SW1.7, U1.VOUT, U7.VCC
- removed net CANH: J55.2, J65.2, R6.1, U7.CANH
- removed net CANL: J55.1, J65.1, R6.2, U7.CANL
- removed net N$13: D5.A, SW1.2, SW1.6
- removed net N$14: C17.1, C7.1, C8.1, C9.1, D5.C, R19.2, U3.VS, U3.VS@1
- removed net N$3: J7.1, R11.2, U2.IN+
- removed net VBAT: C33.1, C34.1, C35.1, C36.1, C43.1, C44.1, Q1.D, Q2.D
- new net M1: J5.1, R11.2, U2.IN+
- new net M2: J5.6, Q2.S, Q3.D
- net +3V3: now also 5V.P$1, C2.1, J5.2, R2.2, U1.VOUT; no longer C16.1, J9.1, SW1.1, SW1.5, U7.VIO
- net ENCODER_1: now also J5.3; no longer J9.2
- net ENCODER_2: now also J5.4; no longer J9.3
- net FDCAN2_RX: no longer TP12.P$1, U7.RXD
- net FDCAN2_TX: no longer TP9.P$1, U7.TXD
- net FDCAN_STB: no longer U7.STB
- net GND: now also J5.5; no longer C15.2, C16.2, J9.4, R19.1, U7.GND
- net M_SH2: no longer J7.2, Q2.S, Q3.D
- net VDD: now also C17.1, C33.1, C34.1, C35.1, C36.1, C43.1, C44.1, C7.1, C8.1, C9.1, Q1.D, Q2.D, U3.VS, U3.VS@1; no longer SW1.4, SW1.8
Other:
- note added: "16V"
- note added: "Пересчитать"
- note removed: "25V"
- note removed: "FDCAN - трансивер"
- moved on the sheet: C10, C100, C11, C12, C13, C14, C17, C18, C23, C24, C25, C26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
