File: Main PCB CAD/STM32 control board.sch (EAGLE design)
At the start: 118 parts, among them J1 PJ-063BH, J10 S3B-PH, J11 S3B-PH, J12 S3B-PH, J13 S3B-PH, J14 S6B-PH, J15 DG301-4P, J2 S3B-PH, J3 S4B-PH, J4 S6B-PH, J5 S3B-PH, J6 S10B-PH, J7 S10B-PH, J8 S10B-PH, J9 S10B-PH, SW1 B3F-4055, SW2 B3F-4055, SW3 B3F-4055, SW4 B3F-4055, SW5 B3F-4055, U1 STM32G474, U2 TPS7A19, U3 REF3330, U4 REF3318, U5 ICM_20600, U6 DRV8701VIA, U8 L2293Q, X1 CSTNE

Commit message: components placement for review
Parts:
- removed J1: PJ-063BH, commonly used connectors:PJ-063BH
- removed J11, J12, J13, J2: S3B-PH, con-jst-ph:S3B-PH
- removed J14: S6B-PH, con-jst-ph:S6B-PH
- removed J3: S4B-PH, con-jst-ph:S4B-PH
- added D10, D11, D12, D13, D14, D15, D16, D17, D18, D19, D20, D21, D22, D23, D24, D25, D26, D27, D28, D29, D30, D31, D32, D33, D34, D35, D36, D37, D6, D7, D8, D9: Blue, Semiconductor_devices:LED0805
- added GND_, TP12, TP13, TP14, TP15, TP16, TP17, TP37, TP38, TP6, TP7, TP8, TP9: (no value), testing:TEST_PAD-[1.27MM_SK]
- added J16, J17, J18, J19: B10B-PH, con-jst-ph:B10B-PH
- added J20, J21, J22, J23: B3B-PH, con-jst-ph:B3B-PH
- added NEG, POS: (no value), testing:SMD_PAD
- added RM2, RM3, RM4, RM5, RM6, RM7, RM8, RM9: RES_ARRAY0603, Resistors:RES_ARRAY0603
- added TP18, TP19, TP20, TP21, TP22, TP23, TP24, TP25, TP26, TP27, TP28, TP29, TP30, TP31, TP32, TP33, TP34, TP35, TP36: (no value), testing:TEST_RING
- J10: value S3B-PH -> B6B-PH; device con-jst-ph:S3B-PH -> con-jst-ph:B6B-PH
- J4: value S6B-PH -> PC_1733570; device con-jst-ph:S6B-PH -> Terminal blocks:PC_1733570
- J5: value S3B-PH -> PC_1733570; device con-jst-ph:S3B-PH -> Terminal blocks:PC_1733570
- J6, J7: value S10B-PH -> B3B-PH; device con-jst-ph:S10B-PH -> con-jst-ph:B3B-PH
- J8: value S10B-PH -> B4B-PH; device con-jst-ph:S10B-PH -> con-jst-ph:B4B-PH
- J9: value S10B-PH -> B6B-PH; device con-jst-ph:S10B-PH -> con-jst-ph:B6B-PH
- RM1: value RES_ARRAY0402_YAGEO -> RES_ARRAY0603; device Resistors:RES_ARRAY0402_YAGEO -> Resistors:RES_ARRAY0603
Connections:
- removed net POUT1: J15.1, U8.OUT1
- removed net POUT2: J15.2, U8.OUT2
- removed net POUT3: J15.3, U8.OUT3
- removed net POUT4: J15.4, U8.OUT4
- new net N$10: D30.C, RM4_4.1
- new net N$12: D27.C, RM4_1.1
- new net N$13: D31.C, RM5_1.1
- new net N$14: D32.C, RM5_2.1
- new net N$22: D34.C, RM5_4.1
- new net N$23: D35.C, RM2_1.1
- new net N$25: D36.C, RM2_2.1
- new net N$26: D14.C, RM2_3.1
- new net N$27: D15.C, RM2_4.1
- new net N$28: D24.C, RM3_1.1
- new net N$29: D25.C, RM3_2.1
- new net N$3: D28.C, RM4_2.1
- new net N$30: D26.C, RM3_3.1
- new net N$31: D37.C, RM3_4.1
- new net N$34: D6.C, RM6_1.1
- new net N$35: D10.C, RM6_2.1
- new net N$36: D7.C, RM6_3.1
- new net N$38: D11.C, RM6_4.1
- new net N$39: D8.C, RM7_1.1
- new net N$40: D12.C, RM7_2.1
- new net N$41: D9.C, RM7_3.1
- new net N$42: D13.C, RM7_4.1
- new net N$43: D16.C, RM8_1.1
- new net N$44: D20.C, RM8_2.1
- new net N$45: D17.C, RM8_3.1
- new net N$46: D21.C, RM8_4.1
- new net N$47: D18.C, RM9_1.1
- new net N$48: D22.C, RM9_2.1
- new net N$49: D19.C, RM9_3.1
- new net N$50: D23.C, RM9_4.1
- new net N$9: D29.C, RM4_3.1
- new net PO1: J15.4, J5.2, TP33.P$1, U8.OUT1
- new net PO2: J15.1, J5.1, TP34.P$1, U8.OUT2
- new net PO3: J15.2, J4.2, TP35.P$1, U8.OUT3
- new net PO4: J15.3, J4.1, TP36.P$1, U8.OUT4
- net +3V: now also J20.1, J21.1, J22.1, J23.1, TP12.P$1, TP15.P$1, TP6.P$1, TP9.P$1
- net +3V3: now also C44.1, J10.2, J16.1, J17.1, J18.1, J19.1, U8.VSS; no longer J10.1, J11.1, J12.1, J13.1, J14.2, J3.1, J4.1, J6.1, J7.1
- net ENCODER_1: now also J10.3, TP30.P$1; no longer J14.3
- net ENCODER_2: now also J10.4, TP29.P$1; no longer J14.4
- net GND: now also GND_.P$1, J10.5, J16.2, J17.2, J18.2, J19.2, J20.3, J21.3, J22.3, J23.3, J6.3, J7.3, J8.4, J9.6, NEG.P, RM1_1.2, RM1_2.2, RM1_3.2, RM1_4.2, RM2_1.2, RM2_2.2, RM2_3.2, RM2_4.2, RM3_1.2, RM3_2.2, RM3_3.2, RM3_4.2, RM4_1.2, RM4_2.2, RM4_3.2, RM4_4.2, RM5_1.2, RM5_2.2, RM5_3.2, RM5_4.2, RM6_1.2, RM6_2.2, RM6_3.2, RM6_4.2, RM7_1.2, RM7_2.2, RM7_3.2, RM7_4.2, RM8_1.2, RM8_2.2, RM8_3.2, RM8_4.2, RM9_1.2, RM9_2.2, RM9_3.2, RM9_4.2, TP14.P$1, TP17.P$1, TP20.P$1, TP21.P$1, TP26.P$1, TP32.P$1, TP8.P$1; no longer D2.C, D3.C, D4.C, D5.C, J1.2, J1.SHIELD, J10.3, J11.3, J12.3, J13.3, J14.5, J2.3, J3.4, J4.6, J5.3, J6.2, J7.2, J8.2, J9.2, TP10.P$1
- net I2C3_SCL: now also J6.2, TP27.P$1; no longer J5.2
- net I2C3_SDA: now also J6.1, TP28.P$1; no longer J5.1
- net M1: now also J10.1, TP31.P$1; no longer J14.1
- net M_SH2: now also J10.6; no longer J14.6
- net N$11: now also D5.C, RM1_4.1; no longer D2.A, RM1_1.2
- net N$17: now also D33.C, RM5_3.1; no longer C44.1, U8.VSS
- net N$19: now also TP37.P$1
- net N$20: now also TP38.P$1
- net N$4: now also D2.C, RM1_1.1; no longer D5.A, RM1_4.2
- net N$5: now also D3.C, RM1_2.1; no longer D4.A, RM1_3.2
- net N$6: now also D4.C, RM1_3.1; no longer D3.A, RM1_2.2
- net PA0: now also J20.2, TP7.P$1; no longer J10.2
- net PA1: now also J21.2, TP10.P$1; no longer J11.2
- net PA2: now also J22.2, TP13.P$1; no longer J12.2
- net PA3: now also J23.2, TP16.P$1; no longer J13.2
- net PB1: now also D4.A; no longer RM1_3.1
- net PB2: now also D5.A; no longer RM1_4.1
- net PC6: now also D2.A; no longer RM1_1.1
- net PC7: now also D3.A; no longer RM1_2.1
- net PD0: now also D27.A, J19.3; no longer J6.3
- net PD1: now also D28.A, J19.4; no longer J6.4
- net PD10: now also D14.A, J16.5; no longer J7.5
- net PD11: now also D15.A, J16.6; no longer J7.6
- net PD12: now also D24.A, J16.7; no longer J7.7
- net PD13: now also D25.A, J16.8; no longer J7.8
- net PD14: now also D26.A, J16.9; no longer J7.9
- net PD15: now also D37.A, J16.10; no longer J7.10
- net PD2: now also D29.A, J19.5; no longer J6.5
- net PD3: now also D30.A, J19.6; no longer J6.6
- net PD4: now also D31.A, J19.7; no longer J6.7
- net PD5: now also D32.A, J19.8; no longer J6.8
- net PD6: now also D33.A, J19.9; no longer J6.9
- net PD7: now also D34.A, J19.10; no longer J6.10
- net PD8: now also D35.A, J16.3; no longer J7.3
- net PD9: now also D36.A, J16.4; no longer J7.4
- net PE0: now also D6.A, J17.3; no longer J8.3
- net PE1: now also D10.A, J17.4; no longer J8.4
- net PE10: now also D17.A, J18.5; no longer J9.5
- net PE11: now also D21.A, J18.6; no longer J9.6
- net PE12: now also D18.A, J18.7; no longer J9.7
- net PE13: now also D22.A, J18.8; no longer J9.8
- net PE14: now also D19.A, J18.9; no longer J9.9
- net PE15: now also D23.A, J18.10; no longer J9.10
- net PE2: now also D7.A, J17.5; no longer J8.5
- net PE3: now also D11.A, J17.6; no longer J8.6
- net PE4: now also D8.A, J17.7; no longer J8.7
- net PE5: now also D12.A, J17.8; no longer J8.8
- net PE6: now also D9.A, J17.9; no longer J8.9
- net PE7: now also D13.A, J17.10; no longer J8.10
- net PE8: now also D16.A, J18.3; no longer J9.3
- net PE9: now also D20.A, J18.4; no longer J9.4
- net SPI3_MISO: now also J9.3, TP24.P$1; no longer J4.3
- net SPI3_MOSI: now also J9.2, TP25.P$1; no longer J4.2
- net SPI3_SCK: now also J9.4, TP23.P$1; no longer J4.4
- net SPI_CS: now also J9.5, TP22.P$1; no longer J4.5
- net SWCLK: now also J8.3; no longer J3.3
- net SWDIO: now also J8.2; no longer J3.2
- net USART3_RX: now also J7.2, TP19.P$1; no longer J2.2
- net USART3_TX: now also J7.1, TP18.P$1; no longer J2.1
- net VDD: now also POS.P; no longer J1.1
Other:
- moved on the sheet: C1, C2, C3, C4, C44, C45, C46, C47, C48, C49, C50, C6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

Commit message: Not finished consept
Parts:
- removed D2, D3, D4, D5: Blue, Semiconductor_devices:LED0805
- removed RM1: RES_ARRAY0603, Resistors:RES_ARRAY0603
Connections:
- removed net N$13: D31.C, RM5_1.1
- removed net N$14: D32.C, RM5_2.1
- removed net N$17: D33.C, RM5_3.1
- removed net N$22: D34.C, RM5_4.1
- removed net PB1: D4.A, U1A.PB1
- removed net PB2: D5.A, U1A.PB2
- removed net PC6: D2.A, U1A.PC6
- removed net PC7: D3.A, U1A.PC7
- net GND: no longer RM1_1.2, RM1_2.2, RM1_3.2, RM1_4.2
- net N$10: now also D34.C, RM5_1.1; no longer D30.C, RM4_4.1
- net N$11: now also D28.C, RM4_3.1; no longer D5.C, RM1_4.1
- net N$12: now also RM4_4.1; no longer RM4_1.1
- net N$3: now also D30.C, RM4_1.1; no longer D28.C, RM4_2.1
- net N$4: now also D31.C, RM5_4.1; no longer D2.C, RM1_1.1
- net N$5: now also D32.C, RM5_3.1; no longer D3.C, RM1_2.1
- net N$6: now also D33.C, RM5_2.1; no longer D4.C, RM1_3.1
- net N$9: now also RM4_2.1; no longer RM4_3.1
Other:
- moved on the sheet: D27, D28, D29, D30, D31, D32, D33, D34

Commit message: consept update
Connections:
- net N$10: now also D28.C, RM4_2.1; no longer D34.C, RM5_1.1
- net N$11: now also D29.C; no longer D28.C
- net N$12: now also D30.C; no longer D27.C
- net N$3: now also D34.C, RM5_4.1; no longer D30.C, RM4_1.1
- net N$4: now also D33.C, RM5_3.1; no longer D31.C, RM5_4.1
- net N$5: now also RM5_2.1; no longer RM5_3.1
- net N$6: now also D31.C, RM5_1.1; no longer D33.C, RM5_2.1
- net N$9: now also D27.C, RM4_1.1; no longer D29.C, RM4_2.1
Other:
- moved on the sheet: D27, D28, D29, D30, D31, D32, D33, D34

Commit message: placement fixes.
Current size is 104*120mm
Parts:
- removed J4, J5: PC_1733570, Terminal blocks:PC_1733570
- removed TP1, TP18, TP19, TP2, TP20, TP21, TP22, TP23, TP24, TP25, TP26, TP27, TP28, TP29, TP3, TP30, TP31, TP32, TP33, TP34, TP35, TP36: (no value), testing:TEST_RING
- removed TP10, TP11, TP12, TP13, TP14, TP15, TP16, TP17, TP6, TP7, TP8, TP9: (no value), testing:TEST_PAD-[1.27MM_SK]
- added J1: B3B-PH, con-jst-ph:B3B-PH
- added JP1: (no value), commonly used connectors:PINHD-1X4
- added JP10, JP4, JP5, JP6, JP7, JP8, JP9: (no value), commonly used connectors:PINHD-1X3
- added JP2, JP3: (no value), commonly used connectors:PINHD-1X6-OCT
Connections:
- removed net PC13: C26.1, R11.1, SW4.1, SW4.2, U1A.PC13
- removed net PC14: C27.1, R12.1, SW5.1, SW5.2, U1A.PC14-OSC32_IN
- new net PB12: C26.1, R11.1, SW4.1, SW4.2, U1A.PB12
- new net PB13: C24.1, R9.1, SW2.1, SW2.2, U1A.PB13
- net +3V: now also JP4.1, JP7.1, JP8.1, JP9.1; no longer TP12.P$1, TP15.P$1, TP6.P$1, TP9.P$1
- net +3V3: now also J1.2, JP10.2, JP2.2, JP3.1; no longer TP1.P$1
- net ENCODER_1: now also JP2.3; no longer TP30.P$1
- net ENCODER_2: now also JP2.4; no longer TP29.P$1
- net GND: now also J1.3, JP10.3, JP2.5, JP3.6, JP4.3, JP5.3, JP6.3, JP7.3, JP8.3, JP9.3, RM2_1.1, RM2_2.1, RM2_3.1, RM2_4.1, RM3_1.1, RM3_2.1, RM3_3.1, RM3_4.1, RM4_1.1, RM4_2.1, RM4_3.1, RM4_4.1, RM5_1.1, RM5_2.1, RM5_3.1, RM5_4.1, RM6_1.1, RM6_2.1, RM6_3.1, RM6_4.1, RM7_1.1, RM7_2.1, RM7_3.1, RM7_4.1, RM8_1.1, RM8_2.1, RM8_3.1, RM8_4.1, RM9_1.1, RM9_2.1, RM9_3.1, RM9_4.1; no longer RM2_1.2, RM2_2.2, RM2_3.2, RM2_4.2, RM3_1.2, RM3_2.2, RM3_3.2, RM3_4.2, RM4_1.2, RM4_2.2, RM4_3.2, RM4_4.2, RM5_1.2, RM5_2.2, RM5_3.2, RM5_4.2, RM6_1.2, RM6_2.2, RM6_3.2, RM6_4.2, RM7_1.2, RM7_2.2, RM7_3.2, RM7_4.2, RM8_1.2, RM8_2.2, RM8_3.2, RM8_4.2, RM9_1.2, RM9_2.2, RM9_3.2, RM9_4.2, TP11.P$1, TP14.P$1, TP17.P$1, TP20.P$1, TP21.P$1, TP26.P$1, TP3.P$1, TP32.P$1, TP8.P$1
- net I2C3_SCL: now also JP5.2; no longer TP27.P$1
- net I2C3_SDA: now also JP5.1; no longer TP28.P$1
- net M1: now also JP2.1; no longer TP31.P$1
- net M_SH2: now also JP2.6
- net N$10: now also RM4_2.2; no longer RM4_2.1
- net N$11: now also RM4_3.2; no longer RM4_3.1
- net N$12: now also RM4_4.2; no longer RM4_4.1
- net N$23: now also RM2_1.2; no longer RM2_1.1
- net N$25: now also RM2_2.2; no longer RM2_2.1
- net N$26: now also RM2_3.2; no longer RM2_3.1
- net N$27: now also RM2_4.2; no longer RM2_4.1
- net N$28: now also RM3_1.2; no longer RM3_1.1
- net N$29: now also RM3_2.2; no longer RM3_2.1
- net N$3: now also RM5_4.2; no longer RM5_4.1
- net N$30: now also RM3_3.2; no longer RM3_3.1
- net N$31: now also RM3_4.2; no longer RM3_4.1
- net N$34: now also RM6_1.2; no longer RM6_1.1
- net N$35: now also RM6_2.2; no longer RM6_2.1
- net N$36: now also RM6_3.2; no longer RM6_3.1
- net N$38: now also RM6_4.2; no longer RM6_4.1
- net N$39: now also RM7_1.2; no longer RM7_1.1
- net N$4: now also RM5_3.2; no longer RM5_3.1
- net N$40: now also RM7_2.2; no longer RM7_2.1
- net N$41: now also RM7_3.2; no longer RM7_3.1
- net N$42: now also RM7_4.2; no longer RM7_4.1
- net N$43: now also RM8_1.2; no longer RM8_1.1
- net N$44: now also RM8_2.2; no longer RM8_2.1
- net N$45: now also RM8_3.2; no longer RM8_3.1
- net N$46: now also RM8_4.2; no longer RM8_4.1
- net N$47: now also RM9_1.2; no longer RM9_1.1
- net N$48: now also RM9_2.2; no longer RM9_2.1
- net N$49: now also RM9_3.2; no longer RM9_3.1
- net N$5: now also RM5_2.2; no longer RM5_2.1
- net N$50: now also RM9_4.2; no longer RM9_4.1
- net N$6: now also RM5_1.2; no longer RM5_1.1
- net N$9: now also RM4_1.2; no longer RM4_1.1
- net PA0: now also JP9.2; no longer TP7.P$1
- net PA1: now also JP8.2; no longer TP10.P$1
- net PA2: now also JP7.2; no longer TP13.P$1
- net PA3: now also JP4.2; no longer TP16.P$1
- net PB14: now also C27.1, R12.1, SW5.1, SW5.2; no longer C24.1, R9.1, SW2.1, SW2.2
- net PO1: now also JP1.1; no longer J5.2, TP33.P$1
- net PO2: now also JP1.2; no longer J5.1, TP34.P$1
- net PO3: now also JP1.3; no longer J4.2, TP35.P$1
- net PO4: now also JP1.4; no longer J4.1, TP36.P$1
- net SPI3_MISO: now also JP3.3; no longer TP24.P$1
- net SPI3_MOSI: now also JP3.2; no longer TP25.P$1
- net SPI3_SCK: now also JP3.4; no longer TP23.P$1
- net SPI_CS: now also JP3.5; no longer TP22.P$1
- net USART3_RX: now also JP6.2; no longer TP19.P$1
- net USART3_TX: now also JP6.1; no longer TP18.P$1
- net VDD: now also J1.1, JP10.1; no longer TP2.P$1
Other:
- moved on the sheet: C6, C7, GND_, J15, TP4, U3

Commit message: routing
Parts:
- removed JP10: (no value), commonly used connectors:PINHD-1X3
Connections:
- removed net M1: J10.1, JP2.1, R13.2, U7.IN+
- new net M2: J10.6, JP2.6, R13.2, U7.IN-
- net +3V3: no longer JP10.2
- net BRIDGE1_EN: now also U1A.PC6; no longer U1B.PF9
- net BRIDGE2_EN: now also U1A.PC7; no longer U1B.PF10
- net GND: no longer JP10.3
- net M_SH1: now also J10.1, JP2.1; no longer R13.1, U7.IN-
- net M_SH2: now also R13.1, U7.IN+; no longer J10.6, JP2.6
- net PO2: now also J15.3; no longer J15.1
- net PO4: now also J15.1; no longer J15.3
- net VDD: no longer JP10.1
Other:
- moved on the sheet: C10, C11, C12, C13, C14, C15, C16, C17, C18, C19, C20, C21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
