File: Main PCB CAD/STM32 control board.sch (EAGLE design)
At the start: 165 parts, among them J1 B3B-PH, J10 B3B-PH, J11 B3B-PH, J12 B3B-PH, J13 B3B-PH, J14 B6B-PH, J15 DG301-4P, J2 B3B-PH, J3 B4B-PH, J4 B6B-PH, J5 B3B-PH, J6 B10B-PH, J7 B10B-PH, J8 B10B-PH, J9 B10B-PH, SW1 B3F-4055, SW2 B3F-4055, SW3 B3F-4055, SW4 B3F-4055, SW5 B3F-4055, U1 STM32G474, U2 TPS7A19, U3 REF3330, U4 REF3318, U5 ICM_20600, U6 DRV8701VIA, U8 L2293Q, X1 CSTNE

Commit message: silkscreen
Parts:
- renumbered PAD1 to POS, PAD2 to NEG
Changed lines of the file:
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@@
 <setting verticaltext="up"/>
 </settings>
-<grid distance="0.1" unitdist="inch" unit="inch" style="lines" multiple="1" display="yes" altdistance="0.01" altunitdist="inch" altunit="inch"/>
+<grid distance="0.1" unitdist="inch" unit="mm" style="lines" multiple="1" display="yes" altdistance="0.01" altunitdist="inch" altunit="inch"/>
 <layers>
 <layer number="1" name="Top" color="4" fill="1" visible="no" active="no"/>
@@
 <part name="D18" library="Semiconductor_devices" library_urn="urn:adsk.eagle:library:13440980" deviceset="LED0805" device="" package3d_urn="urn:adsk.eagle:package:14160208/7" value="Blue"/>
 <part name="D20" library="Semiconductor_devices" library_urn="urn:adsk.eagle:library:13440980" deviceset="LED0805" device="" package3d_urn="urn:adsk.eagle:package:14160208/7" value="Blue"/>
-<part name="PAD1" library="testing" library_urn="urn:adsk.eagle:library:13096589" deviceset="SMD_PAD" device="" package3d_urn="urn:adsk.eagle:package:16041846/4"/>
-<part name="PAD2" library="testing" library_urn="urn:adsk.eagle:library:13096589" deviceset="SMD_PAD" device="" package3d_urn="urn:adsk.eagle:package:16041846/4"/>
+<part name="POS" library="testing" library_urn="urn:adsk.eagle:library:13096589" deviceset="SMD_PAD" device="" package3d_urn="urn:adsk.eagle:package:16041846/4"/>
+<part name="NEG" library="testing" library_urn="urn:adsk.eagle:library:13096589" deviceset="SMD_PAD" device="" package3d_urn="urn:adsk.eagle:package:16041846/4"/>
 <part name="D30" library="Semiconductor_devices" library_urn="urn:adsk.eagle:library:13440980" deviceset="LED0805" device="" package3d_urn="urn:adsk.eagle:package:14160208/7" value="Blue"/>
 <part name="D32" library="Semiconductor_devices" library_urn="urn:adsk.eagle:library:13440980" deviceset="LED0805" device="" package3d_urn="urn:adsk.eagle:package:14160208/7" value="Blue"/>
@@
 <part name="GND33" library="supply1" library_urn="urn:adsk.eagle:library:371" deviceset="GND" device=""/>
 <part name="+3V29" library="supply1" library_urn="urn:adsk.eagle:library:371" deviceset="+3V3" device=""/>
-<part name="J1" library="con-jst-ph" library_urn="urn:adsk.eagle:library:13143856" deviceset="B3B-PH" device="" package3d_urn="urn:adsk.eagle:package:13143941/5"/>
 <part name="TP1" library="testing" library_urn="urn:adsk.eagle:library:13096589" deviceset="TEST_PAD" device="-[1.27MM_SK]" package3d_urn="urn:adsk.eagle:package:15234684/3" value="1.8"/>
 <part name="TP2" library="testing" library_urn="urn:adsk.eagle:library:13096589" deviceset="TEST_PAD" device="-[1.27MM_SK]" package3d_urn="urn:adsk.eagle:package:15234684/3" value="1.8"/>
 <part name="TP3" library="testing" library_urn="urn:adsk.eagle:library:13096589" deviceset="TEST_PAD" device="-[1.27MM_SK]" package3d_urn="urn:adsk.eagle:package:15234684/3" value="1.8"/>
+<part name="J1" library="con-jst-ph" library_urn="urn:adsk.eagle:library:13143856" deviceset="B3B-PH" device="" package3d_urn="urn:adsk.eagle:package:13143941/5"/>
 </parts>
 <sheets>
@@
 <attribute name="VALUE" x="367.03" y="160.02" size="1.778" layer="95"/>
 </instance>
-<instance part="PAD1" gate="1" x="16.51" y="231.14" smashed="yes" grouprefs="POWER_STAGE">
+<instance part="POS" gate="1" x="16.51" y="231.14" smashed="yes" grouprefs="POWER_STAGE">
 <attribute name="NAME" x="15.367" y="232.9942" size="1.778" layer="95"/>
 <attribute name="VALUE" x="15.367" y="227.838" size="1.778" layer="96"/>
 </instance>
-<instance part="PAD2" gate="1" x="16.51" y="226.06" smashed="yes" grouprefs="POWER_STAGE">
+<instance part="NEG" gate="1" x="16.51" y="226.06" smashed="yes" grouprefs="POWER_STAGE">
 <attribute name="NAME" x="15.367" y="227.9142" size="1.778" layer="95"/>
 <attribute name="VALUE" x="15.367" y="222.758" size="1.778" layer="96"/>
@@
 <attribute name="VALUE" x="15.24" y="214.63" size="1.778" layer="96"/>
 </instance>
+<instance part="TP1" gate="G$1" x="96.52" y="158.75" smashed="yes" rot="R270">
+<attribute name="NAME" x="96.52" y="156.21" size="1.27" layer="95" align="center-left"/>
+</instance>
+<instance part="TP2" gate="G$1" x="123.19" y="250.19" smashed="yes" rot="R90">
+<attribute name="NAME" x="123.19" y="252.73" size="1.27" layer="95" rot="R180" align="center-left"/>
+</instance>
+<instance part="TP3" gate="G$1" x="123.19" y="208.28" smashed="yes" rot="R270">
+<attribute name="NAME" x="123.19" y="205.74" size="1.27" layer="95" align="center-left"/>
+</instance>
 <instance part="J1" gate="G$1" x="30.48" y="204.47" smashed="yes">
 <attribute name="VALUE" x="29.21" y="196.85" size="1.778" layer="95"/>
-</instance>
-<instance part="TP1" gate="G$1" x="96.52" y="158.75" smashed="yes" rot="R270">
-<attribute name="NAME" x="96.52" y="156.21" size="1.27" layer="95" align="center-left"/>
-</instance>
-<instance part="TP2" gate="G$1" x="123.19" y="250.19" smashed="yes" rot="R90">
-<attribute name="NAME" x="123.19" y="252.73" size="1.27" layer="95" rot="R180" align="center-left"/>
-</instance>
-<instance part="TP3" gate="G$1" x="123.19" y="208.28" smashed="yes" rot="R270">
-<attribute name="NAME" x="123.19" y="205.74" size="1.27" layer="95" align="center-left"/>
 </instance>
 </instances>
@@
 <wire x1="134.62" y1="219.71" x2="123.19" y2="219.71" width="0.1524" layer="91" grouprefs="POWER_STAGE"/>
 <junction x="123.19" y="219.71" grouprefs="POWER_STAGE"/>
-<pinref part="PAD2" gate="1" pin="P"/>
+<pinref part="NEG" gate="1" pin="P"/>
 <wire x1="27.94" y1="226.06" x2="19.05" y2="226.06" width="0.1524" layer="91" grouprefs="POWER_STAGE"/>
 <pinref part="TP3" gate="G$1" pin="P$1"/>
@@
 <wire x1="17.78" y1="210.82" x2="17.78" y2="204.47" width="0.1524" layer="91"/>
 <pinref part="+3V29" gate="G$1" pin="+3V3"/>
+<wire x1="25.4" y1="204.47" x2="17.78" y2="204.47" width="0.1524" layer="91"/>
 <pinref part="J1" gate="G$1" pin="2"/>
-<wire x1="25.4" y1="204.47" x2="17.78" y2="204.47" width="0.1524" layer="91"/>
 </segment>
 </net>
@@
 <junction x="43.18" y="229.87" grouprefs="POWER_STAGE"/>
 <junction x="25.4" y="231.14" grouprefs="POWER_STAGE"/>
-<pinref part="PAD1" gate="1" pin="P"/>
+<pinref part="POS" gate="1" pin="P"/>
 <wire x1="25.4" y1="231.14" x2="19.05" y2="231.14" width="0.1524" layer="91" grouprefs="POWER_STAGE"/>
 </segment>
@@
 <wire x1="22.86" y1="210.82" x2="22.86" y2="207.01" width="0.1524" layer="91"/>
 <pinref part="VDD5" gate="G$1" pin="VDD"/>
+<wire x1="22.86" y1="207.01" x2="25.4" y2="207.01" width="0.1524" layer="91"/>
 <pinref part="J1" gate="G$1" pin="1"/>
-<wire x1="22.86" y1="207.01" x2="25.4" y2="207.01" width="0.1524" layer="91"/>
-</segment>
-</net>
+</segment>
+</net>

Commit message: silkscreen first time uploaded
Parts:
- removed $1_148_$_2020-08-01_13-42-32: (no value), testing:TEST_PAD-[1.27MM_SK]
- removed TP2, TP3: 1.8, testing:TEST_PAD-[1.27MM_SK]
- removed TP4: 3.0, testing:TEST_PAD-[1.27MM_SK]
- D10, D11, D12, D13, D14, D15, D16, D17, D18, D19, D2, D20, D21, D22, D23, D24, D25, D26, D27, D28, D29, D3, D30, D31, D32, D33, D4, D5, D6, D7, D8, D9: device Semiconductor_devices:LED0805 -> Semiconductor_devices:LED0805CLEAR
- renumbered TP37 to EN1, TP38 to EN2
Connections:
- net N$19 renamed EN1
- net N$20 renamed EN2
- net +3V: no longer TP4.P$1
- net +3V3: no longer TP2.P$1
- net GND: no longer $1_148_$_2020-08-01_13-42-32.P$1, TP3.P$1

Commit message: Silkscreen for rewiew
Parts:
- D1: device Semiconductor_devices:LED0805 -> Semiconductor_devices:LED0805CLEAR
Connections:
- net N$10: now also RM8_2.2; no longer RM1_2.2
- net N$11: now also RM8_3.2; no longer RM1_3.2
- net N$12: now also RM8_4.2; no longer RM1_4.2
- net N$23: now also RM6_1.2; no longer RM5_1.2
- net N$25: now also RM6_2.2; no longer RM5_2.2
- net N$26: now also RM6_3.2; no longer RM5_3.2
- net N$27: now also RM6_4.2; no longer RM5_4.2
- net N$28: now also RM5_1.2; no longer RM7_1.2
- net N$29: now also RM5_2.2; no longer RM7_2.2
- net N$3: now also RM7_4.2; no longer RM3_4.2
- net N$30: now also RM5_3.2; no longer RM7_3.2
- net N$31: now also RM5_4.2; no longer RM7_4.2
- net N$34: now also RM1_1.2; no longer RM2_1.2
- net N$35: now also RM1_2.2; no longer RM2_2.2
- net N$36: now also RM1_3.2; no longer RM2_3.2
- net N$38: now also RM1_4.2; no longer RM2_4.2
- net N$39: now also RM2_1.2; no longer RM4_1.2
- net N$4: now also RM7_3.2; no longer RM3_3.2
- net N$40: now also RM2_2.2; no longer RM4_2.2
- net N$41: now also RM2_3.2; no longer RM4_3.2
- net N$42: now also RM2_4.2; no longer RM4_4.2
- net N$43: now also RM3_1.2; no longer RM6_1.2
- net N$44: now also RM3_2.2; no longer RM6_2.2
- net N$45: now also RM3_3.2; no longer RM6_3.2
- net N$46: now also RM3_4.2; no longer RM6_4.2
- net N$47: now also RM4_1.2; no longer RM8_1.2
- net N$48: now also RM4_2.2; no longer RM8_2.2
- net N$49: now also RM4_3.2; no longer RM8_3.2
- net N$5: now also RM7_2.2; no longer RM3_2.2
- net N$50: now also RM4_4.2; no longer RM8_4.2
- net N$6: now also RM7_1.2; no longer RM3_1.2
- net N$9: now also RM8_1.2; no longer RM1_1.2
Other:
- moved on the sheet: RM1_1, RM1_2, RM1_3, RM1_4, RM2_1, RM2_2, RM2_3, RM2_4, RM3_1, RM3_2, RM3_3, RM3_4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
