File: Main PCB CAD/STM32 control board - ESCD.sch (EAGLE design)
At the start: 161 parts, among them J1 B3B-PH, J10 B3B-PH, J11 B3B-PH, J12 B3B-PH, J13 B3B-PH, J14 B6B-PH, J15 DG301-4P, J2 B3B-PH, J3 B4B-PH, J4 B6B-PH, J5 B3B-PH, J6 B10B-PH, J7 B10B-PH, J8 B10B-PH, J9 B10B-PH, SW1 B3F-4055, SW2 B3F-4055, SW3 B3F-4055, SW4 B3F-4055, SW5 B3F-4055, U1 STM32G474, U2 TPS7A19, U3 REF3330, U4 REF3318, U5 ICM_20600, U6 DRV8701VIA, U8 L2293Q, X1 CSTNE

Commit message: ESCD
Parts:
- removed C49: 10uF, Capacitors:C-EU-CERAMIC1206
- removed C50: 100nF, Capacitors:C-EU-CERAMIC0402
- removed D33: Blue, Semiconductor_devices:LED0805CLEAR
- removed EN1, EN2: (no value), testing:TEST_PAD-[1.27MM_SK]
- removed J1, J10, J11, J12, J13, J2, J5: B3B-PH, con-jst-ph:B3B-PH
- removed J14, J4: B6B-PH, con-jst-ph:B6B-PH
- removed J15: DG301-4P, Terminal blocks:DG301-4P
- removed J3: B4B-PH, con-jst-ph:B4B-PH
- removed J6, J7, J8, J9: B10B-PH, con-jst-ph:B10B-PH
- removed JP1, JP3, JP4, JP5, JP6, JP7: (no value), commonly used connectors:PINHD-1X3
- removed JP2, JP8: (no value), commonly used connectors:PINHD-1X6-OCT
- removed JP9: (no value), commonly used connectors:PINHD-1X4
- removed NEG, POS: (no value), testing:SMD_PAD
- removed Q1, Q2, Q3, Q4: (no value), Transistors:CSD15571Q2
- removed RM1, RM2, RM3, RM4, RM5, RM6, RM7, RM8: RES_ARRAY0603, Resistors:RES_ARRAY0603
- removed TP1, TP5: 1.8, testing:TEST_PAD-[1.27MM_SK]
- removed U1: STM32G474, stmicroelectronics:STM32G4_LPQFP100
- removed U2: TPS7A19, LDOs:TPS7A1901DRBTSON8
- removed U3: REF3330, Voltage references:REF33
- removed U4: REF3318, Voltage references:REF33
- removed U5: ICM_20600, InvenSence:ICM_20600
- removed U6: DRV8701VIA, Transistors drivers:DRV8701VIA
- removed U7: (no value), Current sensing:INA240_TSSOP
- removed U8: L2293Q, Transistors drivers:L2293Q
- removed X1: CSTNE, resonators and oscillators:CSTNE
- added DA1: ESCD_LDOSON8, ESCD:ESCD_LDOSON8
- added DA2, DA3: (no value), ESCD:ESCD_REF
- added DA4: (no value), ESCD:INA240_TSSOP
- added DD1: ICM_20600, ESCD:ICM_20600
- added DD2: ESCD_STM32G4_LPQFP100, ESCD:ESCD_STM32G4_LPQFP100
- added DD3: L2293Q, ESCD:L2293Q
- added DD4: DRV8701, ESCD:DRV8701
- added G1: CSTNE, ESCD:CSTNE
- added R23, R24, R25, R26, R27, R28, R29, R30, R31, R32, R33, R38, R39, R40, R41, R42, R43, R46, R48, R52, R53: ESCD_RES, ESCD:ESCD_RES
- added R34: 16k9, ESCD:ESCD_RES
- added R35, R36, R37, R44, R45: 10k, ESCD:ESCD_RES
- added R47, R49, R50, R51: ESCD_RES_POT, ESCD:ESCD_RES_POT
- added VT1, VT2, VT3, VT4: MOSFET_GOST, ESCD:MOSFET_GOST
- added XS1, XS10, XS12, XS2, XS3, XS4: ESCD_CONNECTOR_3POS, ESCD:ESCD_CONNECTOR_3POS
- added XS11: ESCD_CONNECTOR_2POS, ESCD:ESCD_CONNECTOR_2POS
- added XS13, XS14: ESCD_CONNECTOR_4POS, ESCD:ESCD_CONNECTOR_4POS
- added XS15, XS9: ESCD_CONNECTOR_6POS, ESCD:ESCD_CONNECTOR_6POS
- added XS5, XS6, XS7, XS8: ESCD_CONNECTOR_10POS, ESCD:ESCD_CONNECTOR_10POS
- C1, C30, C33, C38, C4: value 10uF -> ESCD_CAP; device Capacitors:C-EU-CERAMIC1206 -> ESCD:ESCD_CAP; MANUFACTURER_PART_NUMBER CL31B106KAHNNNE -> (none)
- C10, C12, C13, C14, C20, C21, C26, C27, C31, C32, C37, C39, C42, C43, C44, C5: value 100nF -> ESCD_CAP; device Capacitors:C-EU-CERAMIC0402 -> ESCD:ESCD_CAP
- C11, C6, C7, C9: value 4.7uF -> ESCD_CAP; device Capacitors:C-EU-CERAMIC0603 -> ESCD:ESCD_CAP
- C15, C19: value 100nF -> 22uF; device Capacitors:C-EU-CERAMIC0402 -> ESCD:ESCD_CAP
- C16, C17, C24, C25: device Capacitors:C-EU-CERAMIC0402 -> ESCD:ESCD_CAP
- C18, C36, C40, C41: value 1uF -> ESCD_CAP; device Capacitors:C-EU-CERAMIC0603 -> ESCD:ESCD_CAP
- C2, C28, C29, C3, C34, C35, C45, C46, C47, C48: value 22uF -> ESCD_CAP; device Capacitors:C-EU-CERAMIC1210 -> ESCD:ESCD_CAP; MANUFACTURER_PART_NUMBER GRM32ER61C476ME15L -> (none)
- C22, C8: value 4.7uF -> 10uF; device Capacitors:C-EU-CERAMIC0603 -> ESCD:ESCD_CAP
- C23: value 10nF -> ESCD_CAP; device Capacitors:C-EU-CERAMIC0402 -> ESCD:ESCD_CAP
- D1: value Green -> ESCD_LED; device Semiconductor_devices:LED0805CLEAR -> ESCD:ESCD_LED
- D10, D11, D12, D13, D14, D15, D16, D17, D18, D19, D2, D20, D21, D22, D23, D24, D25, D26, D27, D28, D29, D3, D30, D31, D32, D4, D5, D6, D7, D8, D9: value Blue -> ESCD_LED; device Semiconductor_devices:LED0805CLEAR -> ESCD:ESCD_LED
- R1: value 16k9 -> ESCD_RES; device Resistors:R-EU0402 -> ESCD:ESCD_RES
- R10, R11, R12, R14, R15, R2, R3, R4, R9: value 10k -> ESCD_RES; device Resistors:R-EU0402 -> ESCD:ESCD_RES
- R13: value 10 mOhm -> ESCD_RES; device Resistors:R_EU_CS -> ESCD:ESCD_RES; MANUFACTURER_PART_NUMBER ERJ6CWDR010V -> (none)
- R16: value 510k -> ESCD_RES; device Resistors:R-EU0402 -> ESCD:ESCD_RES
- R17, R18, R19, R20, R21, R22: value 100 -> ESCD_RES; device Resistors:R-EU0402 -> ESCD:ESCD_RES
- R5, R6, R7, R8: value 10K -> ESCD_RES; device Resistors:POTEMTIOMETER_EULONG -> ESCD:ESCD_RES
- SW1, SW2, SW3, SW4, SW5: device buttons and switches:B3F-4055 -> ESCD:B3F-4055
Connections:
- removed net +1.8V: C42.1, C9.1, TP5.P$1, U4.OUT, U7.REF1, U7.REF2
- removed net +3V: C10.1, C7.1, J10.1, J11.1, J12.1, J13.1, JP4.1, JP5.1, JP6.1, JP7.1, R5.1, R6.1, R7.1, R8.1, U1C.VREF+, U3.OUT
- removed net AVDD1: C40.2, U6.AVDD, U6.VREF
- removed net BRIDGE1_EN: R21.1, U1A.PC6
- removed net BRIDGE2_EN: R22.1, U1A.PC7
- removed net DRV2_SNSOUT: R15.1, U6.SNSOUT
- removed net DVDD2: C41.2, R14.2, R15.2, U6.DVDD
- removed net EN1: EN1.P$1, R21.2, U8.EN1
- removed net EN2: EN2.P$1, R22.2, U8.EN2
- removed net ENCODER_1: J14.3, JP8.3, U1A.PB4
- removed net ENCODER_2: J14.4, JP8.4, U1A.PB5
- removed net I2C3_SCL: J5.2, JP3.2, U1A.PC8
- removed net I2C3_SDA: J5.1, JP3.1, U1A.PC9
- removed net ICM_CS: U1A.PA4, U5.!CS
- removed net ICM_INT1: U1A.PC4, U5.INT1
- removed net ICM_INT2: U1A.PC5, U5.INT2
- removed net ICM_MISO: U1A.PA6, U5.AD0/SDO
- removed net ICM_MOSI: U1A.PA7, U5.SDA/SDI
- removed net ICM_SCK: U1A.PA5, U5.SCL/SCLK
- removed net M2: J14.6, JP8.6, R13.2, U7.IN-
- removed net MOTOR_CS: U1A.PB0, U7.OUT
- removed net M_GH1: Q1.G, U6.GH1
- removed net M_GH2: Q2.G, U6.GH2
- removed net M_GL1: Q3.G, U6.GL1
- removed net M_GL2: Q4.G, U6.GL2
- removed net M_IN1: U1A.PB6, U6.PH_IN1
- removed net M_IN2: U1A.PB7, U6.EN_IN2
- removed net M_NFAULT: R14.1, U1A.PB9, U6.FAULT_N
- removed net M_NSLEEP: U1A.PB3, U6.SLEEP_N
- removed net M_SH1: J14.1, JP8.1, Q1.S, Q3.D, U6.SH1
- removed net M_SH2: Q2.S, Q4.D, R13.1, U6.SH2, U7.IN+
- removed net N$10: D4.C, RM8_2.2
- removed net N$11: D6.C, RM8_3.2
- removed net N$15: R18.2, U8.IN2
- removed net N$16: R19.2, U8.IN3
- removed net N$18: R20.2, U8.IN4
- removed net N$24: C37.1, U6.CPH
- removed net N$3: D16.C, RM7_4.2
- removed net N$32: C37.2, U6.CPL
- removed net N$33: C36.2, U6.VCP
- removed net N$37: R16.2, U6.IDRIVE
- removed net N$45: D23.C, RM3_3.2
- removed net N$5: D12.C, RM7_2.2
- removed net N$6: D10.C, RM7_1.2
- removed net N$8: R17.2, U8.IN1
- removed net N$9: D2.C, RM8_1.2
- removed net PA0: J10.2, JP4.2, U1A.PA0
- removed net PA1: J11.2, JP5.2, U1A.PA1
- removed net PA2: J12.2, JP6.2, U1A.PA2
- removed net PA3: J13.2, JP7.2, U1A.PA3
- removed net PB12: C26.1, R11.1, SW4.1, SW4.2, U1A.PB12
- removed net PB13: C24.1, R9.1, SW2.1, SW2.2, U1A.PB13
- removed net PB14: C27.1, R12.1, SW5.1, SW5.2, U1A.PB14
- removed net PB15: C25.1, R10.1, SW3.1, SW3.2, U1A.PB15
- removed net PC0: R5.2, U1A.PC0
- removed net PC1: R6.2, U1A.PC1
- removed net PC2: R7.2, U1A.PC2
- removed net PC3: R8.2, U1A.PC3
- removed net PD0: D2.A, J6.3, U1A.PD0
- removed net PD1: D4.A, J6.4, U1A.PD1
- removed net PD10: D22.A, J7.5, U1A.PD10
- removed net PD11: D24.A, J7.6, U1A.PD11
- removed net PD12: D26.A, J7.7, U1A.PD12
- removed net PD13: D28.A, J7.8, U1A.PD13
- removed net PD14: D30.A, J7.9, U1A.PD14
- removed net PD15: D32.A, J7.10, U1A.PD15
- removed net PD2: D6.A, J6.5, U1A.PD2
- removed net PD3: D8.A, J6.6, U1A.PD3
- removed net PD4: D10.A, J6.7, U1A.PD4
- removed net PD5: D12.A, J6.8, U1A.PD5
- removed net PD6: D14.A, J6.9, U1A.PD6
- removed net PD7: D16.A, J6.10, U1A.PD7
- removed net PD8: D18.A, J7.3, U1A.PD8
- removed net PD9: D20.A, J7.4, U1A.PD9
- removed net PE0: D3.A, J8.3, U1B.PE0
- removed net PE1: D5.A, J8.4, U1B.PE1
- removed net PE10: D23.A, J9.5, U1B.PE10
- removed net PE11: D25.A, J9.6, U1B.PE11
- removed net PE12: D27.A, J9.7, U1B.PE12
- removed net PE13: D29.A, J9.8, U1B.PE13
- removed net PE14: D31.A, J9.9, U1B.PE14
- removed net PE15: D33.A, J9.10, U1B.PE15
- removed net PE2: D7.A, J8.5, U1B.PE2
- removed net PE3: D9.A, J8.6, U1B.PE3
- removed net PE4: D11.A, J8.7, U1B.PE4
- removed net PE5: D13.A, J8.8, U1B.PE5
- removed net PE6: D15.A, J8.9, U1B.PE6
- removed net PE7: D17.A, J8.10, U1B.PE7
- removed net PE8: D19.A, J9.3, U1B.PE8
- removed net PE9: D21.A, J9.4, U1B.PE9
- removed net PO1: J15.1, JP9.1, U8.OUT1
- removed net PO2: J15.2, JP9.2, U8.OUT2
- removed net PO3: J15.3, JP9.3, U8.OUT3
- removed net PO4: J15.4, JP9.4, U8.OUT4
- removed net POWER_OUT1: R17.1, U1A.PA8
- removed net POWER_OUT2: R18.1, U1A.PA9
- removed net POWER_OUT3: R19.1, U1A.PA10
- removed net POWER_OUT4: R20.1, U1A.PA11
- removed net REG: C20.1, U5.REGOUT
- removed net RST: C5.1, R3.2, SW1.1, SW1.2, U1B.PG10-NRST
- removed net SPI3_MISO: J4.3, JP2.3, U1A.PC11
- removed net SPI3_MOSI: J4.2, JP2.2, U1A.PC12
- removed net SPI3_SCK: J4.4, JP2.4, U1A.PC10
- removed net SWCLK: J3.3, U1A.PA14
- removed net SWDIO: J3.2, U1A.PA13
- removed net USART3_RX: J2.2, JP1.2, U1A.PB11
- removed net USART3_TX: J2.1, JP1.1, U1A.PB10
- removed net VDD: C1.1, C28.1, C29.1, C30.1, C31.1, C32.1, C33.1, C34.1, C35.1, C36.1, C38.1, C39.1, C45.1, C46.1, C47.1, C48.1, C49.1, C50.1, J1.1, POS.P, Q1.D, Q2.D, U2.EN, U2.VIN, U6.VM, U8.VS, U8.VS@1
- new net 1: XS12.1
- new net 2: XS12.2, XS9.2
- new net 3: XS12.3, XS13.4, XS15.3, XS9.3
- new net 4: XS9.4
- new net 5: XS9.5
- new net 6: XS9.6
- new net B$1: C16.1, C17.1, C24.1, C25.1, DD2.PB12, DD2.PB13, DD2.PB14, DD2.PB15, DD2.PC0, DD2.PC1, DD2.PC2, DD2.PC3, R36.1, R37.1, R44.1, R45.1, R49.3, R50.3, R51.3, SW2.2, SW3.1, SW3.2, SW4.1, SW4.2, SW5.1, SW5.2
- new net E1: DD2.PB4
- new net E2: DD2.PB5, XS15.4
- new net I2S_SCL: DD2.PC8
- new net I2S_SDA: DD2.PC9
- new net N$100: C11.1, R33.1, SW1.1, SW1.2
- new net N$101: DD4.GH1, VT3.P$3
- new net N$102: DD2.PC14
- new net N$103: DD2.PC15
- new net N$104: C27.2, DD4.VCP
- new net N$105: C28.2, DD4.CPL
- new net N$106: C28.1, DD4.CPH
- new net N$107: DD4.GH2, VT1.P$3
- new net N$108: C21.1, DD4.AVDD, DD4.VREF
- new net N$109: C23.1, DD4.DVDD, R46.2, R48.2
- new net N$110: DD4.SNSOUT, R48.1
- new net N$111: DD2.PB9, DD4.FAULT_N, R46.1
- new net N$112: DD4.IDRIVE, R52.2
- new net N$113: DD4.SO
- new net N$114: DD4.GL1, VT2.P$3
- new net N$115: R47.3
- new net N$116: DA4.IN-, DD4.SH2, R53.1, VT3.P$1, VT4.P$2, XS15.6
- new net N$117: DA4.IN+, DD4.SH1, R53.2, VT1.P$1, VT2.P$2, XS15.1
- new net N$118: DD4.GL2, VT4.P$3
- new net N$13: D18.K, R18.1
- new net N$14: D19.K, R19.1
- new net N$17: D20.K, R20.1
- new net N$19: D21.K, R21.1
- new net N$20: D22.K, R22.1
- new net N$22: D23.K, R23.1
- new net N$51: D24.K, R24.1
- new net N$52: D25.K, R25.1
- new net N$53: D26.K, R26.1
- new net N$54: D27.K, R27.1
- new net N$55: D28.K, R28.1
- new net N$56: D29.K, R29.1
- new net N$57: D30.K, R30.1
- new net N$58: D31.K, R31.1
- new net N$59: D32.K, R32.1
- new net N$61: DD3.OUT1, XS14.1
- new net N$62: DD3.OUT3, XS14.3
- new net N$63: DD3.OUT4, XS14.4
- new net N$64: DD2.PB6, DD4.EN_IN2
- new net N$65: DD3.EN1, R42.2
- new net N$66: DD3.IN3, R41.2
- new net N$67: DD3.IN1, R38.2
- new net N$68: DD3.IN2, R39.2
- new net N$69: DD2.PB2
- new net N$70: DD3.IN4, R40.2
- new net N$71: DD2.PB1
- new net N$72: DD2.PB3, DD4.SLEEP_N
- new net N$73: DD2.PB7, DD4.PH_IN1
- new net N$74: DA4.OUT, DD2.PB0
- new net N$76: D1.K, R1.1
- new net N$77: D2.K, R2.1
- new net N$78: D3.K, R3.1
- new net N$79: D4.K, R4.1
- new net N$80: D5.K, R5.1
- new net N$81: D6.K, R6.1
- new net N$82: D7.K, R7.1
- new net N$83: D8.K, R8.1
- new net N$84: D9.K, R9.1
- new net N$85: D10.K, R10.1
- new net N$86: D11.K, R11.1
- new net N$87: D12.K, R12.1
- new net N$88: D13.K, R13.1
- new net N$89: D14.K, R14.1
- new net N$90: D15.K, R15.1
- new net N$91: D16.K, R16.1
- new net N$92: D1.A, D10.A, D11.A, D12.A, D13.A, D14.A, D15.A, D16.A, D2.A, D3.A, D4.A, D5.A, D6.A, D7.A, D8.A, D9.A, DD2.PD0, DD2.PD1, DD2.PD10, DD2.PD11, DD2.PD12, DD2.PD13, DD2.PD14, DD2.PD15, DD2.PD2, DD2.PD3, DD2.PD4, DD2.PD5, DD2.PD6, DD2.PD7, DD2.PD8, DD2.PD9, XS5.10, XS5.3, XS5.4, XS5.5, XS5.6, XS5.7, XS5.8, XS5.9, XS7.10, XS7.3, XS7.4, XS7.5, XS7.6, XS7.7, XS7.8, XS7.9
- new net N$93: DD2.PF1, G1.IN
- new net N$94: DD2.PF0, G1.OUT
- new net N$95: DD2.PF2
- new net N$96: DD2.PF9
- new net N$97: DD2.PF10
- new net N$98: C11.2, DD2.PG10, SW1.3, SW1.4
- new net SPI_MISO: DD2.PC11
- new net SPI_MOSI: DD2.PC12
- new net SPI_SCK: DD2.PC10
- new net UART_RX: DD2.PB11, XS10.2
- new net UART_TX: DD2.PB10, XS10.1
- new net VCC: C1.1, C10.1, C12.1, C13.1, C14.1, C15.1, C18.1, C19.1, C2.1, C20.1, C22.1, C26.1, C27.1, C29.1, C3.1, C30.1, C31.1, C33.1, C34.1, C36.1, C37.1, C39.1, C4.1, C41.1, C42.1, C43.1, C45.1, C5.1, C7.1, C8.1, C9.1, DA1.VIN, DA1.VOUT, DA2.IN, DA2.OUT, DA3.IN, DA3.OUT, DA4.REF1, DA4.REF2, DA4.VS, DD1.VDD, DD1.VDDIO, DD2.VBAT, DD2.VDD, DD2.VDDA, DD2.VDD_2, DD2.VDD_3, DD2.VDD_4, DD2.VDD_5, DD2.VREF+, DD3.VS, DD3.VSS, DD4.VM, R33.2, R34.2, R47.2, R49.2, R50.2, R51.2, XS1.1, XS11.1, XS13.1, XS15.2, XS2.1, XS3.1, XS4.1, XS6.1, XS7.1, XS8.1, XS9.1
- new net VCC1: C32.1, C35.1, C38.1, C40.1, C44.1, C46.1, C47.1, C48.1, VT1.P$2, VT3.P$2
- net +3V3: now also R36.2, R37.2, R44.2, R45.2; no longer C11.1, C12.1, C13.1, C14.1, C15.1, C16.1, C17.1, C18.1, C19.1, C2.1, C21.1, C22.1, C23.1, C3.1, C4.1, C43.1, C44.1, C6.1, C8.1, J1.2, J14.2, J3.1, J4.1, J6.1, J7.1, J8.1, J9.1, JP2.1, JP8.2, R1.2, R10.2, R11.2, R12.2, R3.1, R4.2, R9.2, U1C.VBAT, U1C.VDD, U1C.VDDA, U1C.VDD_2, U1C.VDD_3, U1C.VDD_4, U1C.VDD_5, U2.VOUT, U3.IN, U4.IN, U5.VDD, U5.VDDIO, U7.VS, U8.VSS
- net GND: now also C36.2, C37.2, C40.2, C41.2, DA1.GND, DA1.GND_2, DA1.PAD, DA2.GND, DA3.GND, DA4.GND, DD1.GND, DD1.RESV, DD2.PB8, DD3.GND, DD4.GND, DD4.GND_2, DD4.PAD, DD4.SN, DD4.SP, G1.GND, R1.2, R10.2, R11.2, R12.2, R13.2, R14.2, R15.2, R16.2, R17.2, R18.2, R19.2, R2.2, R20.2, R21.2, R22.2, R23.2, R24.2, R25.2, R26.2, R27.2, R28.2, R29.2, R3.2, R30.2, R31.2, R32.2, R35.1, R4.2, R47.1, R49.1, R5.2, R50.1, R51.1, R52.1, R6.2, R7.2, R8.2, R9.2, VT2.P$1, VT4.P$1, XS1.3, XS10.3, XS11.2, XS15.5, XS2.3, XS3.3, XS4.3, XS6.2, XS7.2, XS8.2; no longer C1.2, C11.2, C12.2, C14.2, C2.2, C27.2, C28.2, C3.2, C4.2, C40.1, C41.1, C49.2, C5.2, C50.2, C7.2, D1.C, J1.3, J10.3, J11.3, J12.3, J13.3, J14.5, J2.3, J3.4, J4.6, J5.3, J6.2, J7.2, J8.2, J9.2, JP1.3, JP2.6, JP3.3, JP4.3, JP5.3, JP6.3, JP7.3, JP8.5, NEG.P, Q3.S, Q4.S, R16.1, R2.1, R5.3, R6.3, R7.3, R8.3, RM1_1.1, RM1_2.1, RM1_3.1, RM1_4.1, RM2_1.1, RM2_2.1, RM2_3.1, RM2_4.1, RM3_1.1, RM3_2.1, RM3_3.1, RM3_4.1, RM4_1.1, RM4_2.1, RM4_3.1, RM4_4.1, RM5_1.1, RM5_2.1, RM5_3.1, RM5_4.1, RM6_1.1, RM6_2.1, RM6_3.1, RM6_4.1, RM7_1.1, RM7_2.1, RM7_3.1, RM7_4.1, RM8_1.1, RM8_2.1, RM8_3.1, RM8_4.1, SW1.3, SW1.4, TP1.P$1, U1A.PB8-BOOT0, U1C.VSS, U1C.VSSA, U1C.VSS_2, U1C.VSS_3, U1C.VSS_4, U1C.VSS_5, U2.GND, U2.GND_2, U2.PAD, U3.GND, U4.GND, U5.GND, U5.RESV, U6.GND, U6.GND_2, U6.PAD, U6.SN, U6.SP, U7.GND, U8.GND, U8.GND@1, U8.GND@2, U8.GND@3, U8.GND@4, U8.NC1@2, U8.NC1@3, U8.NC1@4, U8.NC1@5, U8.NC1@6, U8.NC1@7, U8.NC1@8, U8.NC2@1, U8.NC2@18, U8.NC2@19, U8.NC2@20, U8.NC2@21, U8.NC2@22, U8.NC2@23, X1.GND
- net N$1: now also DD2.PA3, XS1.2; no longer U1B.PF0-OSC_IN, X1.OUT
- net N$12: now also DD2.PA2, XS2.2; no longer D8.C, RM8_4.2
- net N$2: now also XS5.1; no longer U1B.PF1-OSC_OUT, X1.IN
- net N$21: now also DA1.FB, R34.1, R35.2; no longer R1.1, R2.2, U2.FB
- net N$23: now also DD1.INT1, DD2.PC4; no longer D18.C, RM6_1.2
- net N$25: now also DD1.INT2, DD2.PC5; no longer D20.C, RM6_2.2
- net N$26: now also C1.2, C12.2, C14.2, C2.2, C3.2, C4.2, C5.2, C7.2, DD2.VSS, DD2.VSSA, DD2.VSS_2, DD2.VSS_3, DD2.VSS_4, DD2.VSS_5; no longer D22.C, RM6_3.2
- net N$27: now also DD1.!CS, DD2.PA4; no longer D24.C, RM6_4.2
- net N$28: now also DD1.SCL/SCLK, DD2.PA5; no longer D26.C, RM5_1.2
- net N$29: now also DD1.AD0/SDO, DD2.PA6; no longer D28.C, RM5_2.2
- net N$30: now also DD1.SDA/SDI, DD2.PA7; no longer D30.C, RM5_3.2
- net N$31: now also DD2.PA8, R38.1; no longer D32.C, RM5_4.2
- net N$34: now also DD2.PA9, R39.1; no longer D3.C, RM1_1.2
- net N$35: now also D17.A, D18.A, D19.A, D20.A, D21.A, D22.A, D23.A, D24.A, D25.A, D26.A, D27.A, D28.A, D29.A, D30.A, D31.A, D32.A, DD2.PE0, DD2.PE1, DD2.PE10, DD2.PE11, DD2.PE12, DD2.PE13, DD2.PE14, DD2.PE15, DD2.PE2, DD2.PE3, DD2.PE4, DD2.PE5, DD2.PE6, DD2.PE7, DD2.PE8, DD2.PE9, XS6.10, XS6.3, XS6.4, XS6.5, XS6.6, XS6.7, XS6.8, XS6.9, XS8.10, XS8.3, XS8.4, XS8.5, XS8.6, XS8.7, XS8.8, XS8.9; no longer D5.C, RM1_2.2
- net N$36: now also DD2.PA11, R40.1; no longer D7.C, RM1_3.2
- net N$38: now also DD2.PA12; no longer D9.C, RM1_4.2
- net N$39: now also XS13.2; no longer D11.C, RM2_1.2
- net N$4: now also DD2.PC13; no longer D14.C, RM7_3.2
- net N$40: now also DD2.PA14, XS13.3; no longer D13.C, RM2_2.2
- net N$41: now also DD2.PA10, R41.1; no longer D15.C, RM2_3.2
- net N$42: now also DD2.PA0, XS4.2; no longer D17.C, RM2_4.2
- net N$43: now also DD2.PA1, XS3.2; no longer D19.C, RM3_1.2
- net N$44: now also XS5.2; no longer D21.C, RM3_2.2
- net N$46: now also C6.1, DD1.REGOUT; no longer D25.C, RM3_4.2
- net N$47: now also DD3.EN2, R43.2; no longer D27.C, RM4_1.2
- net N$48: now also DD2.PC6, R42.1; no longer D29.C, RM4_2.2
- net N$49: now also DD2.PC7, R43.1; no longer D31.C, RM4_3.2
- net N$50: now also DD3.OUT2, XS14.2; no longer D33.C, RM4_4.2
- net N$7: now also D17.K, R17.1; no longer D1.A, R4.1
- net SPI_CS: now also DD2.PA15; no longer J4.5, JP2.5, U1A.PA15
Other:
- note added: "+1V8"
- note added: "+3V0"
- note added: "+3V3"
- note added: "1"
- note added: "10"
- note added: "11"
- note added: "12"
- note added: "13"
- note added: "14"
- note added: "15"
- note added: "16"
- note added: "2"
- note added: "3"
- note added: "4"
- note added: "5"
- note added: "6"
- note added: "7"
- note added: "8"
- note added: "9"
- note added: "E1"
- note added: "E2"
- note added: "GND"
- note added: "I2C_SCL"
- note added: "I2C_SDA"
- note added: "M1"
- note added: "M2"
- note added: "PD0"
- note added: "PD1"
- note added: "PD10"
- note added: "PD11"
- note added: "PD12"
- note added: "PD13"
- note added: "PD14"
- note added: "PD15"
- note added: "PD2"
- note added: "PD3"
- note added: "PD4"
- note added: "PD5"
- note added: "PD6"
- note added: "PD7"
- note added: "PD8"
- note added: "PD9"
- note added: "PE0"
- note added: "PE1"
- note added: "PE10"
- note added: "PE11"
- note added: "PE12"
- note added: "PE13"
- note added: "PE14"
- note added: "PE15"
- note added: "PE2"
- note added: "PE3"
- note added: "PE4"
- note added: "PE5"
- note added: "PE6"
- note added: "PE7"
- note added: "PE8"
- note added: "PE9"
- note added: "P_OUT1"
- note added: "P_OUT2"
- note added: "P_OUT3"
- note added: "P_OUT4"
- note added: "SPI_CS"
- note added: "SPI_MISO"
- note added: "SPI_MOSI"
- note added: "SPI_SCK"
- note added: "SWCLK"
- note added: "SWIDO"
- note added: "Sensor1"
- note added: "Sensor2"
- note added: "Sensor3"
- note added: "Sensor4"
- note added: "UART_RX"
- note added: "UART_TX"
- note added: "Vin"
- note added: "БГУИР, каф. СУ"
- note added: "ГУИР.ХХХХХХ.001 Э3"
- note added: "Плата управления стендом STM32"
- note added: "Схема электрическая принципиальная"
- note removed: "16V"
- note removed: "Calculated output voltage is 3.317 V. Tolerance of resistors in FB voltage divider is 1%"
- note removed: "Grid size 0.05 inch, Alt 0.01 inch"
- note removed: "Schematic designed to work either from external power adapter (from 12V to 5V) or from ST-Link 3.3V power line"
- note removed: "VDD 1-5 и VBAT"
- note removed: "VDDA"
