File: Extention board/ESCD.sch (EAGLE design)
At the start: 31 parts

Commit message: ESCD
Parts:
- renumbered A to D1, B to D2, C to D3, D to D4, E to D5, F to D6, G to D7, H to D8
Connections:
- net GND: now also R15.1, R3.1, R4.1; no longer R10.1, R12.1, R14.1
- net N$1: now also R5.2; no longer R1.2
- net N$13: now also R1.2, R3.2; no longer R10.2, R9.2
- net N$14: now also R1.1, R14.1, R2.1; no longer R11.1, R15.1, R9.1
- net N$15: now also R13.2, R15.2, VT3.P$3; no longer R11.2, R12.2, VT2.P$3
- net N$16: now also R2.2, R4.2, VT2.P$3; no longer R13.2, R14.2, VT3.P$3
- net N$17: now also R14.2; no longer R15.2
- net N$2: now also R6.2; no longer R2.2
- net N$21: now also R12.2; no longer R8.2
- net N$3: now also R7.2; no longer R3.2
- net N$4: now also R8.2; no longer R4.2
- net N$5: now also R9.2; no longer R5.2
- net N$6: now also R10.2; no longer R6.2
- net N$7: now also R11.2; no longer R7.2
- net N$76: now also R5.1; no longer R1.1
- net N$77: now also R6.1; no longer R2.1
- net N$78: now also R7.1; no longer R3.1
- net N$79: now also R8.1; no longer R4.1
- net N$80: now also R9.1; no longer R5.1
- net N$81: now also R10.1; no longer R6.1
- net N$82: now also R11.1; no longer R7.1
- net N$83: now also R12.1; no longer R8.1
Other:
- note added: "Плата модуля расширения"
- note removed: "Плата управления стендом STM32"
- moved on the sheet: R1, R10, R11, R12, R13, R14, R15, R2, R3, R4, R5, R6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
